Commit message: Feat: Simulation Boat

File: simulation/description/dock.urdf.xacro (robot description, xacro)
@@ -11,10 +11,10 @@
     <visual>
       <geometry>
-       <mesh filename="file:///home/username/dev_ws/src/my_package/meshes/DOCK4.dae"/>
+       <mesh filename="file:///home/username/dev_ws/src/simulation/meshes/DOCK4.dae"/>
       </geometry>
     </visual>
     <collision name="base_link_collision">
       <geometry>
-       <mesh filename="file:///home/username/dev_ws/src/my_package/meshes/DOCK4.dae"/>
+       <mesh filename="file:///home/username/dev_ws/src/simulation/meshes/DOCK4.dae"/>
       </geometry>
     </collision>
@@ -41,5 +41,5 @@
             <origin xyz="0 0 0.1" rpy="1.5708 0 1.5708"/>
             <geometry>
-                <mesh filename="file:///home/username/dev_ws/src/my_package/meshes/terminal.dae" scale="0.001 0.001 0.001"/>
+                <mesh filename="file:///home/username/dev_ws/src/simulation/meshes/terminal.dae" scale="0.001 0.001 0.001"/>
             </geometry>
         </collision>
@@ -47,5 +47,5 @@
             <origin xyz="0 0 0.1" rpy="1.5708 0 1.5708"/>
             <geometry>
-              <mesh filename="file:///home/username/dev_ws/src/my_package/meshes/terminal.dae" scale="0.001 0.001 0.001"/>
+              <mesh filename="file:///home/username/dev_ws/src/simulation/meshes/terminal.dae" scale="0.001 0.001 0.001"/>
             </geometry>
         </visual>
